Commit message: Actually have a nice simulation working using just sin waves to drive robot inputs.

File: urdf/manual_puppet.urdf (robot description, URDF)
Before this commit: robot puppet, 26 links, 25 joints
Links:
- removed link left_elbow_psi_link
- removed link left_knee_psi_link
- removed link right_elbow_psi_link
- removed link right_knee_psi_link
- added link left_elbow_phi_link
- added link left_knee_phi_link
- added link right_elbow_phi_link
- added link right_knee_phi_link
Joints:
- removed joint left_elbow_psi
- removed joint left_knee_psi
- removed joint right_elbow_psi
- removed joint right_knee_psi
- added joint left_elbow_phi: type continuous, parent left_shoulder_phi_link, child left_elbow_phi_link, origin xyz=0.0 0.0 -0.2, axis 1 0 0
- added joint left_knee_phi: type continuous, parent left_hip_phi_link, child left_knee_phi_link, origin xyz=0.0 0.0 -0.35, axis 1 0 0
- added joint right_elbow_phi: type continuous, parent right_shoulder_phi_link, child right_elbow_phi_link, origin xyz=0.0 0.0 -0.2, axis 1 0 0
- added joint right_knee_phi: type continuous, parent right_hip_phi_link, child right_knee_phi_link, origin xyz=0.0 0.0 -0.35, axis 1 0 0
- joint left_radius_connection: parent left_elbow_psi_link -> left_elbow_phi_link
- joint left_tibia_connection: parent left_knee_psi_link -> left_knee_phi_link
- joint right_radius_connection: parent right_elbow_psi_link -> right_elbow_phi_link
- joint right_tibia_connection: parent right_knee_psi_link -> right_knee_phi_link

Commit message: Added markers for all of the strings.  Also added "hook" frames to the urdf.

File: urdf/manual_puppet.urdf (robot description, URDF)
Before this commit: robot puppet, 26 links, 25 joints
Links:
- added link left_hand_hook
- added link left_knee_hook
- added link left_shoulder_hook
- added link right_hand_hook
- added link right_knee_hook
- added link right_shoulder_hook
Joints:
- added joint left_hand_hook_connection: type fixed, parent left_radius, child left_hand_hook, origin xyz=0.0 0.0 -0.2
- added joint left_knee_hook_connection: type fixed, parent left_femur, child left_knee_hook, origin xyz=0.0 -0.038 -0.302
- added joint left_shoulder_hook_connection: type fixed, parent torso, child left_shoulder_hook, origin xyz=0.1632 0.0 0.08352
- added joint right_hand_hook_connection: type fixed, parent right_radius, child right_hand_hook, origin xyz=0.0 0.0 -0.2
- added joint right_knee_hook_connection: type fixed, parent right_femur, child right_knee_hook, origin xyz=0.0 -0.038 -0.302
- added joint right_shoulder_hook_connection: type fixed, parent torso, child right_shoulder_hook, origin xyz=-0.1632 0.0 0.08352
